Commit message: changes updated

File: description/robot.urdf.xacro (robot description, xacro)
@@ -2,3 +2,5 @@
 <robot xmlns:xacro="http://www.ros.org/wiki/xacro"  name="robot">
     <xacro:include filename='robot_core.xacro'/>
+    <xacro:include filename='gazebo_control.xacro'/>
+    <xacro:include filename='lidar.xacro'/>
 </robot>

File: description/robot_core.xacro (robot description, xacro)
@@ -14,4 +14,7 @@
     <material name='black'>
         <color rgba='0 0 0 1'/>
+    </material>
+    <material name="red">
+        <color rgba="1 0 0 1"/>
     </material>
     <!-- BASE LINK -->
@@ -38,8 +41,11 @@
             </geometry>
         </collision>
-        <xaro:inertial_box mass='0.5' x='0.3' y='0.3' z='0.15'>
+        <xacro:inertial_box mass='0.5' x='0.3' y='0.3' z='0.15'>
             <origin xyz='0.15 0 0.075' rpy='0 0 0'/>
         </xacro:inertial_box>
     </link>
+    <gazebo reference='chassis'>
+        <material>Gazebo/White</material>
+    </gazebo>
     <!-- LEFT WHEEL LINK -->
     <joint name='left_wheel_joint' type='continuous'>
@@ -61,8 +67,11 @@
             </geometry>
         </collision>
-        <xaro:inertial_cylinder mass='0.1' length='0.04' radius='0.05'>
+        <xacro:inertial_cylinder mass='0.1' length='0.04' radius='0.05'>
             <origin xyz='0 0 0' rpy='0 0 0'/>
         </xacro:inertial_cylinder>
     </link>
+    <gazebo reference='left_wheel'>
+        <material>Gazebo/Blue</material>
+    </gazebo>
     <!-- RIGHT WHEEL LINK -->
     <joint name='right_wheel_joint' type='continuous'>
@@ -84,8 +93,11 @@
             </geometry>
         </collision>
-        <xaro:inertial_cylinder mass='0.1' length='0.04' radius='0.05'>
+        <xacro:inertial_cylinder mass='0.1' length='0.04' radius='0.05'>
             <origin xyz='0 0 0' rpy='0 0 0'/>
         </xacro:inertial_cylinder>
     </link>
+    <gazebo reference='right_wheel'>
+        <material>Gazebo/Blue</material>
+    </gazebo>
     <!-- CASTER WHEEL LINK -->
     <joint name="caster_wheel_joint" type="fixed">
@@ -107,6 +119,11 @@
         </collision>
         <xacro:inertial_sphere mass='0.1' radius='0.05'>
-            <origin xyz='0 0 0' rpy='0 0 0'>
+            <origin xyz='0 0 0' rpy='0 0 0'/>
         </xacro:inertial_sphere>
     </link>
+    <gazebo reference='caster_wheel'>
+        <material>Gazebo/Black</material>
+        <mu1 value='0.001'/>
+        <mu2 value='0.001'/>
+    </gazebo>
 </robot>
